File: battery_monitoring.sch (KiCad schematic (older format))
At the start: 11 parts, among them P1 TC_SWD, SW4 SW_SP3T, U7 STM32F030F4Px

Commit message: Component placement WIP - multiple Hammond enclosures drawn
Parts:
- RN3: footprint (none) -> Resistors_SMD:R_Array_Convex_4x0402
- renumbered RN3 to RN4
Changed lines of the file:
@@
 $EndComp
 $Comp
-L R_Pack04 RN3
+L R_Pack04 RN4
 U 1 1 5AA115B7
 P 7250 4900
-F 0 "RN3" V 6950 4900 50  0000 C CNN
+F 0 "RN4" V 6950 4900 50  0000 C CNN
 F 1 "4*1k" V 7450 4900 50  0000 C CNN
 F 2 "Resistors_SMD:R_Array_Convex_4x0402" V 7525 4900 50  0001 C CNN
@@
 F 0 "RN3" H 10330 2370 50  0000 L CNN
 F 1 "10k" H 10330 2310 50  0000 L CNN
-F 2 "" H 10300 2350 50  0001 C CNN
+F 2 "Resistors_SMD:R_Array_Convex_4x0402" H 10300 2350 50  0001 C CNN
 F 3 "" H 10300 2350 50  0001 C CNN
 	4    10300 2350

Commit message: Almost all components placed... Saving before mirroring everything
Parts:
- removed BAR1: DOT-BAR, Displays:HDSP-48xx, symbol DOT-BAR
- added D10: Red, LEDs:LED_0603, symbol LED_Small
- added D5, D6, D7: Green, LEDs:LED_0603, symbol LED_Small
- added D8, D9: Yellow, LEDs:LED_0603, symbol LED_Small
Connections:
- wire segments 74 -> 64
Other:
- note added: "LED array for battery level display"
- note removed: "Charlieplexed LED bar for battery level display"
- moved on the sheet: RN4

Commit message: v1.0   Add 3D files with Hammond enclosures  fabrication outputs
Parts:
- R15: value 270k 1% -> 270k,1%
- R16: value 31.6k 1% -> 31.6k,1%
- renumbered RN3 to RN2
Connections:
- net 3.3V_EN: now also U7.2 (PF0-OSC_IN/RCC_OSC_IN); no longer U7.13 (PA7/ADC_IN7/SPI1_MOSI/TIM14_CH1/TIM17_CH1/TIM1_CH1N/TIM3_CH2)
- net ESP32_EN: now also U7.13 (PA7/ADC_IN7/SPI1_MOSI/TIM14_CH1/TIM17_CH1/TIM1_CH1N/TIM3_CH2); no longer U7.12 (PA6/ADC_IN6/SPI1_MISO/TIM16_CH1/TIM1_BKIN/TIM3_CH1)
- net MAIN_OUT_EN: now also U7.12 (PA6/ADC_IN6/SPI1_MISO/TIM16_CH1/TIM1_BKIN/TIM3_CH1); no longer U7.2 (PF0-OSC_IN/RCC_OSC_IN)
Other:
- note added: "Li-Po\nLi-Fe\nCustom (set by ESP32)"
- note removed: "Li-Po\nLi-Fe\nSlave"
Changed lines of the file:
@@
 Text Notes 750  5700 0    60   ~ 0
 Battery type selector
+Text HLabel 2900 1550 0    60   Output ~ 0
+MAIN_OUT_EN
 Text HLabel 2900 2650 0    60   Output ~ 0
-MAIN_OUT_EN
-Text HLabel 2900 1650 0    60   Output ~ 0
 3.3V_EN
 Text HLabel 2900 950  0    60   Input ~ 0
 EN_PUSH_BUTTON
-Text HLabel 2900 1550 0    60   Output ~ 0
+Text HLabel 2900 1650 0    60   Output ~ 0
 ESP32_EN
 $Comp
@@
 $EndComp
 $Comp
-L +3.3V #PWR081
+L +3.3V #PWR084
 U 1 1 5AA0E175
 P 2850 3000
-F 0 "#PWR081" H 2850 2850 50  0001 C CNN
+F 0 "#PWR084" H 2850 2850 50  0001 C CNN
 F 1 "+3.3V" H 2850 3140 50  0000 C CNN
 F 2 "" H 2850 3000 50  0001 C CNN
@@
 Connection ~ 3350 3050
 $Comp
-L GND #PWR082
+L GND #PWR085
 U 1 1 5AA0E1F8
 P 2850 3300
-F 0 "#PWR082" H 2850 3050 50  0001 C CNN
+F 0 "#PWR085" H 2850 3050 50  0001 C CNN
 F 1 "GND" H 2850 3150 50  0000 C CNN
 F 2 "" H 2850 3300 50  0001 C CNN
@@
 $EndComp
 $Comp
-L GND #PWR083
+L GND #PWR086
 U 1 1 5AA0E21F
 P 3000 3300
-F 0 "#PWR083" H 3000 3050 50  0001 C CNN
+F 0 "#PWR086" H 3000 3050 50  0001 C CNN
 F 1 "GND" H 3000 3150 50  0000 C CNN
 F 2 "" H 3000 3300 50  0001 C CNN
@@
 $EndComp
 $Comp
-L GND #PWR084
+L GND #PWR087
 U 1 1 5AA0E254
 P 9900 3000
-F 0 "#PWR084" H 9900 2750 50  0001 C CNN
+F 0 "#PWR087" H 9900 2750 50  0001 C CNN
 F 1 "GND" H 9900 2850 50  0000 C CNN
 F 2 "" H 9900 3000 50  0001 C CNN
@@
 USART1 is also used by\nthe serial bootloader.
 $Comp
-L +BATT #PWR085
+L +BATT #PWR088
 U 1 1 5AA0E847
 P 1000 6650
-F 0 "#PWR085" H 1000 6500 50  0001 C CNN
+F 0 "#PWR088" H 1000 6500 50  0001 C CNN
 F 1 "+BATT" H 1000 6790 50  0000 C CNN
 F 2 "" H 1000 6650 50  0001 C CNN
@@
 Battery voltage measurement\n+BATT = 30V => 3.14V
 $Comp
-L GND #PWR086
+L GND #PWR089
 U 1 1 5AA0EDE2
 P 1000 7250
-F 0 "#PWR086" H 1000 7000 50  0001 C CNN
+F 0 "#PWR089" H 1000 7000 50  0001 C CNN
 F 1 "GND" H 1000 7100 50  0000 C CNN
 F 2 "" H 1000 7250 50  0001 C CNN
@@
 P 1000 6800
 F 0 "R15" H 1030 6820 50  0000 L CNN
-F 1 "270k 1%" H 1030 6760 50  0000 L CNN
+F 1 "270k,1%" H 1030 6760 50  0000 L CNN
 F 2 "Resistors_SMD:R_0603" H 1000 6800 50  0001 C CNN
 F 3 "" H 1000 6800 50  0001 C CNN
@@
 P 1000 7100
 F 0 "R16" H 1030 7120 50  0000 L CNN
-F 1 "31.6k 1%" H 1030 7060 50  0000 L CNN
+F 1 "31.6k,1%" H 1030 7060 50  0000 L CNN
 F 2 "Resistors_SMD:R_0603" H 1000 7100 50  0001 C CNN
 F 3 "" H 1000 7100 50  0001 C CNN
@@
 $EndComp
 $Comp
-L GND #PWR087
+L GND #PWR090
 U 1 1 5AA0F425
 P 1250 7250
-F 0 "#PWR087" H 1250 7000 50  0001 C CNN
+F 0 "#PWR090" H 1250 7000 50  0001 C CNN
 F 1 "GND" H 1250 7100 50  0000 C CNN
 F 2 "" H 1250 7250 50  0001 C CNN
@@
 	5700 7050 5750 7050
 $Comp
-L GND #PWR088
+L GND #PWR091
 U 1 1 5AA14FB1
 P 850 5400
-F 0 "#PWR088" H 850 5150 50  0001 C CNN
+F 0 "#PWR091" H 850 5150 50  0001 C CNN
 F 1 "GND" H 850 5250 50  0000 C CNN
 F 2 "" H 850 5400 50  0001 C CNN
@@
 NoConn ~ 1950 2150
 $Comp
-L GND #PWR089
+L GND #PWR092
 U 1 1 5AA18D74
 P 750 2150
-F 0 "#PWR089" H 750 1900 50  0001 C CNN
+F 0 "#PWR092" H 750 1900 50  0001 C CNN
 F 1 "GND" H 750 2000 50  0000 C CNN
 F 2 "" H 750 2150 50  0001 C CNN
@@
 $EndComp
 $Comp
-L +3.3V #PWR090
+L +3.3V #PWR093
 U 1 1 5AA18DFB
 P 750 1950
-F 0 "#PWR090" H 750 1800 50  0001 C CNN
+F 0 "#PWR093" H 750 1800 50  0001 C CNN
 F 1 "+3.3V" H 750 2090 50  0000 C CNN
 F 2 "" H 750 1950 50  0001 C CNN
@@
 NoConn ~ 3450 2750
 Text Notes 2100 5450 0    60   ~ 0
-Li-Po\nLi-Fe\nSlave
-$Comp
-L GND #PWR091
+Li-Po\nLi-Fe\nCustom (set by ESP32)
+$Comp
+L GND #PWR094
 U 1 1 5AA153F7
 P 10300 2450
-F 0 "#PWR091" H 10300 2200 50  0001 C CNN
+F 0 "#PWR094" H 10300 2200 50  0001 C CNN
 F 1 "GND" H 10300 2300 50  0000 C CNN
 F 2 "" H 10300 2450 50  0001 C CNN
@@
 $EndComp
 $Comp
-L GND #PWR092
+L GND #PWR095
 U 1 1 5AA1619D
 P 10150 3050
-F 0 "#PWR092" H 10150 2800 50  0001 C CNN
+F 0 "#PWR095" H 10150 2800 50  0001 C CNN
 F 1 "GND" H 10150 2900 50  0000 C CNN
 F 2 "" H 10150 3050 50  0001 C CNN
@@
 	2900 1450 3450 1450
 $Comp
-L R_Pack04_Unit RN3
+L R_Pack04_Unit RN2
 U 4 1 5AA2FEC7
 P 10300 2350
-F 0 "RN3" H 10330 2370 50  0000 L CNN
+F 0 "RN2" H 10330 2370 50  0000 L CNN
 F 1 "10k" H 10330 2310 50  0000 L CNN
 F 2 "Resistors_SMD:R_Array_Convex_4x0402" H 10300 2350 50  0001 C CNN

Commit message: v1.1 - changed some resistor values ; manufacturability improvements (thermal relief) ; added a test point for ESP32_EN
Parts:
- RN2: value 10k -> 1k
- RN4: value 4*1k -> 4*100R
Changed lines of the file:
@@
 P 5500 6950
 F 0 "RN4" V 5200 6950 50  0000 C CNN
-F 1 "4*1k" V 5700 6950 50  0000 C CNN
+F 1 "4*100R" V 5700 6950 50  0000 C CNN
 F 2 "Resistors_SMD:R_Array_Convex_4x0402" V 5775 6950 50  0001 C CNN
 F 3 "" H 5500 6950 50  0001 C CNN
@@
 P 10300 2350
 F 0 "RN2" H 10330 2370 50  0000 L CNN
-F 1 "10k" H 10330 2310 50  0000 L CNN
+F 1 "1k" H 10330 2310 50  0000 L CNN
 F 2 "Resistors_SMD:R_Array_Convex_4x0402" H 10300 2350 50  0001 C CNN
 F 3 "" H 10300 2350 50  0001 C CNN
