File: KXKM_audio_battery_module.kicad_pcb (KiCad board)
At the start: 2 copper layers, 56.5 x 57.5 mm, 80 parts, among them J1 Conn_01x06, J10 Conn_01x02, J12 Audio-Jack-3, J2 TEST_1P, J3 mikroBUS_socket, J4 Conn_01x04, J5 Micro_SD_Card, J6 Conn_01x03, J7 Conn_01x04, J8 Conn_01x02, J9 Conn_01x05, P1 TC_SWD, Q1 DMN63D8LDW, Q2 DMN63D8LDW, Q3 DMN63D8LDW, SW1 SW_Push, SW2 SW_Push, SW3 SW_Push, SW4 SW_SP3T, U1 ESP32-WROOM, U2 SP3485CN, U3 MCP16331T-E/CH, U4 BTS50080-1TEA, U5 DC_DC_POL, U6 PCM5141, U7 STM32F030F4Px

Commit message: v1.1 - changed some resistor values ; manufacturability improvements (thermal relief) ; added a test point for ESP32_EN
Parts:
- added J11: TEST_1P, Connectors_TestPoints:Test_Point_Pad_d1.5mm, F.Cu at (121.8, 93.2)
- RN2: value 10k -> 1k
- RN4: value 4*1k -> 4*100R
Routing:
- net GND: track 594.2 -> 591.0 mm
- net /ESP32_EN: track 44.8 -> 47.2 mm
- net +BATT: track 73.6 -> 75.9 mm
Other:
- board text added: "DTR"
- board text added: "GND"
- board text added: "Tom Magnier v1.1 04/2018"
- board text added: "v1.1 04/2018"
- board text removed: "Tom Magnier v1.0 03/2018"
- board text removed: "v1.0 03/2018"
Changed lines of the file:
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@@
 (kicad_pcb (version 4) (host pcbnew 4.0.7)
   (general
-    (links 263)
+    (links 270)
     (no_connects 0)
-    (area 102.924999 80.424999 159.575001 138.075001)
+    (area 82.766667 61.2 226.171429 171.95)
     (thickness 1.6)
-    (drawings 86)
-    (tracks 1527)
+    (drawings 88)
+    (tracks 1531)
     (zones 0)
-    (modules 80)
+    (modules 81)
     (nets 92)
   )
@@
   (title_block
     (title "ESP32 Audio & Battery module")
-    (date 2018-03-15)
-    (rev 1.0)
+    (date 2018-03-29)
+    (rev 1.1)
     (company KXKM)
     (comment 1 "Tom Magnier")
@@
     (mod_text_size 1 1)
     (mod_text_width 0.15)
-    (pad_size 1 0.8)
+    (pad_size 6 6)
     (pad_drill 0)
     (pad_to_mask_clearance 0.07)
@@
       (net 4 +BATT))
     (pad 2 smd rect (at 3.05 0) (size 4 2.5) (layers F.Cu F.Paste F.Mask)
-      (net 1 GND))
+      (net 1 GND) (thermal_width 1))
     (model Capacitors_SMD.3dshapes/CP_Elec_8x10.wrl
       (at (xyz 0 0 0))
@@
       (net 1 GND))
     (pad 39 smd rect (at -0.3 -0.5 270) (size 6 6) (layers F.Cu F.Paste F.Mask)
-      (net 1 GND))
+      (net 1 GND) (zone_connect 2))
     (pad 15 smd oval (at -9 9.58) (size 0.9 2.5) (layers F.Cu F.Paste F.Mask)
       (net 1 GND))
@@
       (effects (font (size 1 1) (thickness 0.15)) (justify mirror))
     )
-    (fp_text value 10k (at 0 -2.1 270) (layer B.Fab) hide
+    (fp_text value 1k (at 0 -2.1 270) (layer B.Fab) hide
       (effects (font (size 1 1) (thickness 0.15)) (justify mirror))
     )
@@
       (effects (font (size 1 1) (thickness 0.15)) (justify mirror))
     )
-    (fp_text value 4*1k (at 0 -2.1 180) (layer B.Fab) hide
+    (fp_text value 4*100R (at 0 -2.1 180) (layer B.Fab) hide
       (effects (font (size 1 1) (thickness 0.15)) (justify mirror))
     )
@@
     )
   )
+  (module Connectors_TestPoints:Test_Point_Pad_d1.5mm (layer F.Cu)
+    (at 121.75 93.25)
+    (descr "SMD pad as test Point, diameter 1.5mm")
+    (tags "test point SMD pad")
+    (attr virtual)
+    (fp_text reference J11 (at 0 0) (layer F.Fab)
+      (effects (font (size 1 1) (thickness 0.15)))
+    )
+    (fp_text value TEST_1P (at 0 1.75) (layer F.Fab) hide
+      (effects (font (size 1 1) (thickness 0.15)))
+    )
+    (fp_text user %R (at 0 -1.65) (layer F.Fab) hide
+      (effects (font (size 1 1) (thickness 0.15)))
+    )
+    (fp_circle (center 0 0) (end 1.25 0) (layer F.CrtYd) (width 0.05))
+    (fp_circle (center 0 0) (end 0 0.95) (layer F.SilkS) (width 0.12))
+    (pad 1 smd circle (at 0 0) (size 1.5 1.5) (layers F.Cu F.Mask)
+      (net 2 /ESP32_EN))
+  )
+  (gr_text GND (at 106.25 82.25 270) (layer F.SilkS)
+    (effects (font (size 0.8 0.75) (thickness 0.15)))
+  )
+  (gr_text DTR (at 106.5 95 270) (layer F.SilkS)
+    (effects (font (size 0.8 0.75) (thickness 0.15)))
+  )
   (gr_line (start 128.75 109.25) (end 133.75 109.25) (layer Dwgs.User) (width 0.2))
   (gr_line (start 131.25 106.75) (end 131.25 111.75) (layer Dwgs.User) (width 0.2))
@@
     (arrow2b (pts (xy 103 63) (xy 104.126504 62.413579)))
   )
-  (gr_text "Tom Magnier\nv1.0 03/2018" (at 137.25 95 180) (layer B.SilkS)
+  (gr_text "Tom Magnier\nv1.1 04/2018" (at 137.25 95 180) (layer B.SilkS)
     (effects (font (size 1 1) (thickness 0.2)) (justify mirror))
   )
@@
     (effects (font (size 1.2 1.2) (thickness 0.25)) (justify mirror))
   )
-  (gr_text "v1.0\n03/2018" (at 121 91.5 180) (layer F.SilkS)
+  (gr_text "v1.1\n04/2018" (at 118.75 91.25 180) (layer F.SilkS)
     (effects (font (size 1 1) (thickness 0.2)))
   )
@@
   (gr_circle (center 145.25 95.25) (end 145.25 96.75) (layer Dwgs.User) (width 0.2))
   (gr_circle (center 117.25 95.25) (end 117.25 96.75) (layer Dwgs.User) (width 0.2))
+  (segment (start 117.483276 120.029208) (end 117.483276 120.766724) (width 0.4) (layer F.Cu) (net 1))
+  (segment (start 117.483276 120.766724) (end 117.05 121.2) (width 0.4) (layer F.Cu) (net 1))
+  (segment (start 117.05 121.2) (end 115.913733 121.2) (width 0.4) (layer F.Cu) (net 1))
+  (segment (start 115.913733 121.2) (end 115.823754 121.110021) (width 0.4) (layer F.Cu) (net 1))
+  (segment (start 117.483276 102.029208) (end 117.483276 101.733276) (width 0.4) (layer F.Cu) (net 1))
+  (segment (start 117.483276 101.733276) (end 117 101.25) (width 0.4) (layer F.Cu) (net 1))
+  (segment (start 117 101.25) (end 116.75 101.25) (width 0.4) (layer F.Cu) (net 1))
+  (segment (start 148.075736 92.5) (end 136.75 92.5) (width 1) (layer F.Cu) (net 1))
+  (segment (start 148.5 92.5) (end 148.075736 92.5) (width 0.16) (layer F.Cu) (net 1))
+  (segment (start 148.75 93.25) (end 148.5 93) (width 0.6) (layer F.Cu) (net 1))
+  (segment (start 148.5 93) (end 148.5 92.5) (width 0.6) (layer F.Cu) (net 1))
+  (segment (start 150.95 93.25) (end 148.75 93.25) (width 0.6) (layer F.Cu) (net 1))
+  (segment (start 148.75 93.25) (end 148.5 93.5) (width 0.6) (layer F.Cu) (net 1))
+  (segment (start 148.5 93.5) (end 148.5 94.5) (width 0.6) (layer F.Cu) (net 1))
   (segment (start 140.99 122.5) (end 139.89 123.6) (width 0.16) (layer B.Cu) (net 1))
   (segment (start 133.75 125.004002) (end 133.75 125.442044) (width 0.16) (layer B.Cu) (net 1))
@@
   (segment (start 152.37 121.63) (end 150.8 123.2) (width 0.16) (layer F.Cu) (net 1))
   (via (at 150.8 123.2) (size 0.6) (drill 0.4) (layers F.Cu B.Cu) (net 1))
-  (segment (start 117.483276 120.029208) (end 117.012484 120.5) (width 0.4) (layer F.Cu) (net 1))
-  (segment (start 117.012484 120.5) (end 116.162484 120.5) (width 0.4) (layer F.Cu) (net 1))
-  (segment (start 116.162484 120.5) (end 115.823754 120.83873) (width 0.4) (layer F.Cu) (net 1))
-  (segment (start 115.823754 120.83873) (end 115.823754 121.110021) (width 0.4) (layer F.Cu) (net 1))
   (segment (start 124.29 135.25) (end 125.5 135.25) (width 0.4) (layer B.Cu) (net 1))
   (segment (start 125.5 135.25) (end 125.619999 135.369999) (width 0.4) (layer B.Cu) (net 1))
@@
   (segment (start 150.95 91.7) (end 150.75 91.5) (width 0.6) (layer F.Cu) (net 1))
   (via (at 150.75 91.5) (size 0.6) (drill 0.4) (layers F.Cu B.Cu) (net 1))
-  (segment (start 149.75 92.5) (end 148.5 92.5) (width 1) (layer F.Cu) (net 1))
-  (segment (start 148.5 92.5) (end 136.75 92.5) (width 1) (layer F.Cu) (net 1))
-  (segment (start 150.95 93.25) (end 149.25 93.25) (width 0.6) (layer F.Cu) (net 1))
-  (segment (start 149.25 93.25) (end 148.5 92.5) (width 0.6) (layer F.Cu) (net 1))
   (via (at 148.5 92.5) (size 0.6) (drill 0.4) (layers F.Cu B.Cu) (net 1))
-  (segment (start 150.95 93.25) (end 149.75 93.25) (width 0.6) (layer F.Cu) (net 1))
-  (segment (start 149.75 93.25) (end 148.5 94.5) (width 0.6) (layer F.Cu) (net 1))
   (via (at 148.5 94.5) (size 0.6) (drill 0.4) (layers F.Cu B.Cu) (net 1))
   (segment (start 134 86) (end 135.75 86) (width 0.4) (layer F.Cu) (net 1))
@@
   (segment (start 108.5 96.5) (end 107.75 96.5) (width 0.16) (layer B.Cu) (net 1) (status 10))
   (via (at 107.75 96.5) (size 0.6) (drill 0.4) (layers F.Cu B.Cu) (net 1))
-  (segment (start 117.483276 102.029208) (end 117.483276 101.983276) (width 0.4) (layer F.Cu) (net 1) (status 30))
-  (segment (start 117.483276 101.983276) (end 116.75 101.25) (width 0.4) (layer F.Cu) (net 1) (status 10))
   (via (at 116.75 101.25) (size 0.6) (drill 0.4) (layers F.Cu B.Cu) (net 1))
   (segment (start 108.548961 94) (end 108.15 94) (width 0.16) (layer F.Cu) (net 1) (status 30))
@@
   (via (at 135.75 93.75) (size 0.6) (drill 0.4) (layers F.Cu B.Cu) (net 1))
   (segment (start 150.95 93.25) (end 150.5 93.25) (width 1) (layer F.Cu) (net 1) (status 30))
-  (segment (start 150.5 93.25) (end 149.75 92.5) (width 1) (layer F.Cu) (net 1) (status 30))
   (segment (start 136.75 92.5) (end 136.25 93) (width 1) (layer F.Cu) (net 1))
   (segment (start 134 86) (end 134 88.288788) (width 0.6) (layer F.Cu) (net 1))
@@
   (via (at 135.456908 132.698984) (size 0.6) (drill 0.4) (layers F.Cu B.Cu) (net 1))
   (segment (start 110 92.25) (end 110 92.3) (width 0.16) (layer B.Cu) (net 1) (status 30))
+  (segment (start 121.75 95.272861) (end 121.75 93.25) (width 0.16) (layer F.Cu) (net 2))
+  (segment (start 122.035726 95.558587) (end 121.75 95.272861) (width 0.16) (layer F.Cu) (net 2))
   (segment (start 119.699997 115.972935) (end 119.999996 116.272934) (width 0.16) (layer B.Cu) (net 2))
   (segment (start 118.1 114.372938) (end 119.699997 115.972935) (width 0.16) (layer B.Cu) (net 2))
@@
   (segment (start 132.511909 133.238984) (end 132.166908 133.238984) (width 0.4) (layer B.Cu) (net 3) (status 30))
   (segment (start 132.166908 133.238984) (end 130.206908 135.198984) (width 0.4) (layer B.Cu) (net 3) (status 30))
+  (segment (start 154.75 93.25) (end 157.05 93.25) (width 1) (layer F.Cu) (net 4))
+  (segment (start 157.05 93.25) (end 157.05 94.95) (width 1) (layer F.Cu) (net 4))
   (segment (start 157.05 93.25) (end 154.75 93.25) (width 0.6) (layer B.Cu) (net 4))
   (via (at 154.75 93.25) (size 0.6) (drill 0.4) (layers F.Cu B.Cu) (net 4))
-  (segment (start 157.05 93.25) (end 157.05 94.95) (width 0.6) (layer F.Cu) (net 4))
   (segment (start 157.05 94.95) (end 157 95) (width 0.6) (layer F.Cu) (net 4))
   (via (at 157 95) (size 0.6) (drill 0.4) (layers F.Cu B.Cu) (net 4))
@@
   )
   (zone (net 1) (net_name GND) (layer F.Cu) (hatch edge 0.508)
-    (connect_pads thru_hole_only (clearance 0.2))
+    (connect_pads (clearance 0.2))
     (min_thickness 0.2)
-    (fill yes (arc_segments 16) (thermal_gap 0.2) (thermal_bridge_width 0.5))
+    (fill yes (arc_segments 16) (thermal_gap 0.2) (thermal_bridge_width 0.8))
     (polygon
       (pts

Commit message: Update BOM & fab files
Parts:
- R1, R2: value 10k -> 10k,1%
Changed lines of the file:
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@@
       (effects (font (size 1 1) (thickness 0.15)) (justify mirror))
     )
-    (fp_text value 10k (at 0 -1.5 90) (layer B.Fab) hide
+    (fp_text value 10k,1% (at 0 -1.5 90) (layer B.Fab) hide
       (effects (font (size 1 1) (thickness 0.15)) (justify mirror))
     )
@@
       (effects (font (size 1 1) (thickness 0.15)) (justify mirror))
     )
-    (fp_text value 10k (at 0 -1.5) (layer B.Fab) hide
+    (fp_text value 10k,1% (at 0 -1.5) (layer B.Fab) hide
       (effects (font (size 1 1) (thickness 0.15)) (justify mirror))
     )
