File: Base_board/KXKM_ESP32_battery_management_board.sch (KiCad schematic (older format))
At the start: 38 parts, among them J1 Conn_01x06, J11 TEST_1P, J2 TEST_1P, J3 Conn_02x10_Odd_Even, J4 Conn_01x04, J5 Micro_SD_Card, J6 Conn_01x03, J7 Conn_01x03, J8 Conn_01x03, Q1 BC847W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

Commit message: Fix older symbols assignation
Parts:
- C1, C2, C3: symbol KXKM_audio_battery_module-rescue:C_Small -> Device:C_Small
- J1: symbol KXKM_audio_battery_module-rescue:Conn_01x06 -> Connector_Generic:Conn_01x06
- J11, J2: symbol KXKM_audio_battery_module-rescue:TEST_1P -> Connector:TestPoint
- J4: symbol KXKM_audio_battery_module-rescue:Conn_01x04 -> Connector_Generic:Conn_01x04
- J5: symbol KXKM_audio_battery_module-rescue:Micro_SD_Card -> Connector:Micro_SD_Card
- J6: symbol KXKM_audio_battery_module-rescue:Conn_01x03 -> Connector_Generic:Conn_01x03
- MK1, MK2: symbol KXKM_audio_battery_module-rescue:Mounting_Hole -> Mechanical:MountingHole
- R7: symbol KXKM_audio_battery_module-rescue:R_Small -> Device:R_Small
- SW1: symbol KXKM_audio_battery_module-rescue:SW_Push -> Switch:SW_Push
- U1: symbol KXKM_audio_battery_module-rescue:ESP32-WROOM -> espressif-xess:ESP32-WROOM
- U2: symbol KXKM_audio_battery_module-rescue:SP3485CN -> Interface_UART:SP3485CN
Changed lines of the file:
@@
 EESchema Schematic File Version 4
-LIBS:KXKM_audio_battery_module-cache
+LIBS:KXKM_ESP32_battery_management_board-cache
 EELAYER 29 0
 EELAYER END
@@
 $EndDescr
 $Comp
-L KXKM_audio_battery_module-rescue:ESP32-WROOM U1
+L espressif-xess:ESP32-WROOM U1
 U 1 1 5A8A8AB3
 P 4550 2150
@@
 $EndSheet
 $Comp
-L KXKM_audio_battery_module-rescue:SP3485CN U2
+L Interface_UART:SP3485CN U2
 U 1 1 5A9FA1D2
 P 9500 3500
@@
 $EndComp
 $Comp
-L KXKM_audio_battery_module-rescue:Micro_SD_Card J5
+L Connector:Micro_SD_Card J5
 U 1 1 5A9FA363
 P 9800 1400
@@
 NB : IO15 = MTDO = debug log enabled\nIO0 AND IO2 must be low to enter BL \nIO2 : internal PD, IO0 : internal PU
 $Comp
-L KXKM_audio_battery_module-rescue:GND #PWR01
+L power:GND #PWR01
 U 1 1 5AA001B2
 P 4400 2050
@@
 $EndComp
 $Comp
-L KXKM_audio_battery_module-rescue:GND #PWR02
+L power:GND #PWR02
 U 1 1 5AA004A8
 P 7100 1950
@@
 $EndComp
 $Comp
-L KXKM_audio_battery_module-rescue:GND #PWR03
+L power:GND #PWR03
 U 1 1 5AA00743
 P 5450 4250
@@
 NoConn ~ 6950 2750
 $Comp
-L KXKM_audio_battery_module-rescue:C_Small C2
+L Device:C_Small C2
 U 1 1 5AA00E87
 P 3850 1850
@@
 $EndComp
 $Comp
-L KXKM_audio_battery_module-rescue:GND #PWR04
+L power:GND #PWR04
 U 1 1 5AA015D5
 P 3850 1950
@@
 $EndComp
 $Comp
-L KXKM_audio_battery_module-rescue:+3.3V #PWR05
+L power:+3.3V #PWR05
 U 1 1 5AA0164D
 P 3850 1650
@@
 $EndSheet
 $Comp
-L KXKM_audio_battery_module-rescue:+3.3V #PWR06
+L power:+3.3V #PWR06
 U 1 1 5AA1FF0E
 P 1550 4900
@@
 NoConn ~ 8900 1800
 $Comp
-L KXKM_audio_battery_module-rescue:GND #PWR07
+L power:GND #PWR07
 U 1 1 5AA21253
 P 8400 1750
@@
 $EndComp
 $Comp
-L KXKM_audio_battery_module-rescue:+3.3V #PWR08
+L power:+3.3V #PWR08
 U 1 1 5AA21355
 P 8400 1350
@@
 $EndComp
 $Comp
-L KXKM_audio_battery_module-rescue:GND #PWR09
+L power:GND #PWR09
 U 1 1 5AA216A0
 P 10650 2050
@@
 SD_DO
 $Comp
-L KXKM_audio_battery_module-rescue:+3.3V #PWR010
+L power:+3.3V #PWR010
 U 1 1 5AA22B6F
 P 8150 4900
@@
 DMX / RS-485 transceiver
 $Comp
-L KXKM_audio_battery_module-rescue:GND #PWR011
+L power:GND #PWR011
 U 1 1 5AA23FA0
 P 9500 3900
@@
 $EndComp
 $Comp
-L KXKM_audio_battery_module-rescue:C_Small C3
+L Device:C_Small C3
 U 1 1 5AA25004
 P 9300 2800
@@
 $EndComp
 $Comp
-L KXKM_audio_battery_module-rescue:+3.3V #PWR012
+L power:+3.3V #PWR012
 U 1 1 5AA25178
 P 9300 2700
@@
 $EndComp
 $Comp
-L KXKM_audio_battery_module-rescue:GND #PWR013
+L power:GND #PWR013
 U 1 1 5AA25212
 P 9300 2900
@@
 $EndComp
 $Comp
-L KXKM_audio_battery_module-rescue:R_Small R7
+L Device:R_Small R7
 U 1 1 5AA256B0
 P 10050 3500
@@
 $EndComp
 $Comp
-L KXKM_audio_battery_module-rescue:Conn_01x03 J6
+L Connector_Generic:Conn_01x03 J6
 U 1 1 5AA25B5C
 P 10750 3600
@@
 $EndComp
 $Comp
-L KXKM_audio_battery_module-rescue:GND #PWR014
+L power:GND #PWR014
 U 1 1 5AA25EA0
 P 10500 3750
@@
 DMX_DI
 $Comp
-L KXKM_audio_battery_module-rescue:GND #PWR015
+L power:GND #PWR015
 U 1 1 5AA27614
 P 10000 6050
@@
 Extension connector
 $Comp
-L KXKM_audio_battery_module-rescue:Mounting_Hole MK2
+L Mechanical:MountingHole MK2
 U 1 1 5AA02B66
 P 6550 7650
@@
 $EndComp
 $Comp
-L KXKM_audio_battery_module-rescue:Mounting_Hole MK1
+L Mechanical:MountingHole MK1
 U 1 1 5AA02C9C
 P 5950 7650
@@
 $EndComp
 $Comp
-L KXKM_audio_battery_module-rescue:Conn_01x04 J4
+L Connector_Generic:Conn_01x04 J4
 U 1 1 5AA0E433
 P 6600 6800
@@
 I2C_SDA
 $Comp
-L KXKM_audio_battery_module-rescue:GND #PWR016
+L power:GND #PWR016
 U 1 1 5AA0EF07
 P 6300 6600
@@
 $EndComp
 $Comp
-L KXKM_audio_battery_module-rescue:+3.3V #PWR017
+L power:+3.3V #PWR017
 U 1 1 5AA0F052
 P 6100 6750
@@
 $EndComp
 $Comp
-L KXKM_audio_battery_module-rescue:SW_Push SW1
+L Switch:SW_Push SW1
 U 1 1 5AA13971
 P 1950 2550
@@
 $EndComp
 $Comp
-L KXKM_audio_battery_module-rescue:TEST_1P J2
+L Connector:TestPoint J2
 U 1 1 5AA13BA9
 P 1750 2450
@@
 Tie STM32_BOOT to 3.3V to start UART bootloader.
 $Comp
-L KXKM_audio_battery_module-rescue:GND #PWR018
+L power:GND #PWR018
 U 1 1 5AA165C1
 P 2200 2550
@@
 ESP32_EN
 $Comp
-L KXKM_audio_battery_module-rescue:Conn_01x06 J1
+L Connector_Generic:Conn_01x06 J1
 U 1 1 5AA18902
 P 1150 7000
@@
 Serial & programmation connector with ESP32 auto-reset
 $Comp
-L KXKM_audio_battery_module-rescue:GND #PWR019
+L power:GND #PWR019
 U 1 1 5AA19B5E
 P 2000 6750
@@
 PROG_RTS
 $Comp
-L KXKM_audio_battery_module-rescue:+3.3V #PWR020
+L power:+3.3V #PWR020
 U 1 1 5AA19EC3
 P 2200 6950
@@
 PROG_DTR
 $Comp
-L KXKM_audio_battery_module-rescue:C_Small C1
+L Device:C_Small C1
 U 1 1 5AA1B767
 P 3800 2500
@@
 $EndComp
 $Comp
-L KXKM_audio_battery_module-rescue:GND #PWR021
+L power:GND #PWR021
 U 1 1 5AA1B90F
 P 3800 2600
@@
 Buffer for 5V digital LED strip
 $Comp
-L KXKM_audio_battery_module-rescue:+3.3V #PWR022
+L power:+3.3V #PWR022
 U 1 1 5AA2C62F
 P 8150 5550
@@
 Input only\nNo PU, no PD
 $Comp
-L KXKM_audio_battery_module-rescue:GND #PWR029
+L power:GND #PWR029
 U 1 1 5AA26E5F
 P 6500 1250
@@
 $EndComp
 $Comp
-L KXKM_audio_battery_module-rescue:VBUS #PWR030
+L power:VBUS #PWR030
 U 1 1 5AA7F3B8
 P 9050 4900
@@
 $EndComp
 $Comp
-L KXKM_audio_battery_module-rescue:VBUS #PWR031
+L power:VBUS #PWR031
 U 1 1 5AA7F756
 P 9050 5550
@@
 $EndComp
 $Comp
-L KXKM_audio_battery_module-rescue:VBUS #PWR032
+L power:VBUS #PWR032
 U 1 1 5AA7FB52
 P 10000 5200
@@
 	6950 3450 7550 3450
 $Comp
-L KXKM_audio_battery_module-rescue:TEST_1P J11
+L Connector:TestPoint J11
 U 1 1 5ABD450A
 P 4700 7500
@@
 P/N : 112J-TDAR-R01 / TFP09-2-12B
 $Comp
-L KXKM_audio_battery_module-rescue:GND #PWR0127
+L power:GND #PWR0127
 U 1 1 5CA3FB9A
 P 4000 5550
@@
 LED_DATA_1
 $Comp
-L KXKM_audio_battery_module-rescue:+3.3V #PWR0128
+L power:+3.3V #PWR0128
 U 1 1 5CA40497
 P 3100 4550
@@
 	3100 4600 3200 4600
 $Comp
-L KXKM_audio_battery_module-rescue:+BATT #PWR0103
+L power:+BATT #PWR0103
 U 1 1 5CB8685A
 P 4050 4550
@@
 $EndComp
 $Comp
-L KXKM_audio_battery_module-rescue:VBUS #PWR0104
+L power:VBUS #PWR0104
 U 1 1 5CB8B602
 P 2850 4550
@@
 $EndComp
 $Comp
-L KXKM_audio_battery_module-rescue:GND #PWR0109
+L power:GND #PWR0109
 U 1 1 5CB8E7AB
 P 10000 5400
@@
 $EndComp
 $Comp
-L KXKM_audio_battery_module-rescue:VBUS #PWR0110
+L power:VBUS #PWR0110
 U 1 1 5CB9730E
 P 10000 5850
