File: Base_board/KXKM_ESP32_battery_management_board.sch (KiCad schematic (older format))
At the start: 37 parts, among them J1 Conn_01x06, J11 TEST_1P, J2 TEST_1P, J3 Conn_02x10_Odd_Even, J4 Conn_01x04, J6 Conn_01x03, J7 Conn_01x03, J8 Conn_01x03, Q1 BC847W, Q2 BC847W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

Commit message: rescue from cache
Parts:
- U1: symbol espressif-xess:ESP32-WROOM -> KXKM_ESP32_battery_management_board-rescue:ESP32-WROOM-espressif-xess
Changed lines of the file:
@@
 $EndDescr
 $Comp
-L espressif-xess:ESP32-WROOM U1
+L KXKM_ESP32_battery_management_board-rescue:ESP32-WROOM-espressif-xess U1
 U 1 1 5A8A8AB3
 P 4550 2150

Commit message: update, etc
Parts:
- added R33, R34, R36, R38: 22k, Resistor_SMD:R_0603_1608Metric, symbol Device:R_Small
- added R35, R37: 10k, Resistor_SMD:R_0603_1608Metric, symbol Device:R_Small
- added SW2: SW_DIP_x03, Button_Switch_THT:SW_DIP_SPSTx03_Piano_CTS_Series194-3MSTN_W7.62mm_P2.54mm, symbol Switch:SW_DIP_x03
Connections:
- net +3V3: now also SW2.4, SW2.5, SW2.6
- net GND: now also R33.1
- net DIP_SWITCH: now reaches U1.6 (IO34)
- net DIP_SWITCH: now also R37.2, R38.1
- new net: R33.2, R34.1, R35.1
- new net: R34.2, SW2.1
- new net: R35.2, R36.1, R37.1
- new net: R36.2, SW2.2
- new net: R38.2, SW2.3
- no-connect marks 15 -> 14
Changed lines of the file:
@@
 F4 "EN_PUSH_BUTTON" O L 2050 1100 60
 F5 "LOAD_I_SENSE" O L 2050 1200 60
+F6 "AUTOBOOT_SENSE" O L 2050 1300 60
 $EndSheet
 $Comp
@@
 F9 "STM32_BOOT" I R 1550 2450 60
 F10 "LOAD_I_SENSE" I R 1550 1200 60
+F11 "AUTOBOOT_SENSE" I R 1550 1300 60
 $EndSheet
 $Comp
@@
 	1    1500 7100
 	0    1    1    0
-$EndComp
-$Comp
-L Device:R_Small R4
-U 1 1 5C76546B
-P 1600 5200
-F 0 "R4" H 1541 5154 50  0000 R CNN
-F 1 "10k" H 1541 5245 50  0000 R CNN
-F 2 "Resistor_SMD:R_0603_1608Metric" H 1600 5200 50  0001 C CNN
-F 3 "~" H 1600 5200 50  0001 C CNN
-	1    1600 5200
-	-1   0    0    1
 $EndComp
 $Comp
@@
 Wire Wire Line
 	6950 3150 7550 3150
-NoConn ~ 4550 2650
 Text Label 3950 2850 0    60   ~ 12
 I2C_SDA
@@
 NoConn ~ 7550 2950
 NoConn ~ 7550 2850
+Wire Wire Line
+	1550 1300 2050 1300
+$Comp
+L Switch:SW_DIP_x03 SW2
+U 1 1 613120EE
+P 5900 5500
+F 0 "SW2" H 5900 5967 50  0000 C CNN
+F 1 "SW_DIP_x03" H 5900 5876 50  0000 C CNN
+F 2 "Button_Switch_THT:SW_DIP_SPSTx03_Piano_CTS_Series194-3MSTN_W7.62mm_P2.54mm" H 5900 5500 50  0001 C CNN
+F 3 "~" H 5900 5500 50  0001 C CNN
+	1    5900 5500
+	0    -1   -1   0
+$EndComp
+$Comp
+L Device:R_Small R4
+U 1 1 5C76546B
+P 1600 5200
+F 0 "R4" H 1541 5154 50  0000 R CNN
+F 1 "10k" H 1541 5245 50  0000 R CNN
+F 2 "Resistor_SMD:R_0603_1608Metric" H 1600 5200 50  0001 C CNN
+F 3 "~" H 1600 5200 50  0001 C CNN
+	1    1600 5200
+	-1   0    0    1
+$EndComp
+$Comp
+L Device:R_Small R34
+U 1 1 612F26B9
+P 5475 6025
+F 0 "R34" H 5416 5979 50  0000 R CNN
+F 1 "22k" H 5416 6070 50  0000 R CNN
+F 2 "Resistor_SMD:R_0603_1608Metric" H 5475 6025 50  0001 C CNN
+F 3 "~" H 5475 6025 50  0001 C CNN
+	1    5475 6025
+	-1   0    0    1
+$EndComp
+$Comp
+L Device:R_Small R36
+U 1 1 612F94AC
+P 5800 6025
+F 0 "R36" H 5741 5979 50  0000 R CNN
+F 1 "22k" H 5741 6070 50  0000 R CNN
+F 2 "Resistor_SMD:R_0603_1608Metric" H 5800 6025 50  0001 C CNN
+F 3 "~" H 5800 6025 50  0001 C CNN
+	1    5800 6025
+	-1   0    0    1
+$EndComp
+$Comp
+L Device:R_Small R38
+U 1 1 612F9613
+P 6100 6025
+F 0 "R38" H 6041 5979 50  0000 R CNN
+F 1 "22k" H 6041 6070 50  0000 R CNN
+F 2 "Resistor_SMD:R_0603_1608Metric" H 6100 6025 50  0001 C CNN
+F 3 "~" H 6100 6025 50  0001 C CNN
+	1    6100 6025
+	-1   0    0    1
+$EndComp
+$Comp
+L Device:R_Small R33
+U 1 1 612FB75C
+P 5250 6225
+F 0 "R33" V 5325 6275 50  0000 R CNN
+F 1 "22k" V 5150 6275 50  0000 R CNN
+F 2 "Resistor_SMD:R_0603_1608Metric" H 5250 6225 50  0001 C CNN
+F 3 "~" H 5250 6225 50  0001 C CNN
+	1    5250 6225
+	0    -1   -1   0
+$EndComp
+$Comp
+L Device:R_Small R35
+U 1 1 612FBF19
+P 5650 6225
+F 0 "R35" V 5725 6250 50  0000 R CNN
+F 1 "10k" V 5550 6275 50  0000 R CNN
+F 2 "Resistor_SMD:R_0603_1608Metric" H 5650 6225 50  0001 C CNN
+F 3 "~" H 5650 6225 50  0001 C CNN
+	1    5650 6225
+	0    -1   -1   0
+$EndComp
+$Comp
+L Device:R_Small R37
+U 1 1 6131DE4A
+P 5975 6225
+F 0 "R37" V 6050 6275 50  0000 R CNN
+F 1 "10k" V 5875 6275 50  0000 R CNN
+F 2 "Resistor_SMD:R_0603_1608Metric" H 5975 6225 50  0001 C CNN
+F 3 "~" H 5975 6225 50  0001 C CNN
+	1    5975 6225
+	0    -1   -1   0
+$EndComp
+Wire Wire Line
+	5700 5800 5700 5850
+Wire Wire Line
+	5700 5850 5475 5850
+Wire Wire Line
+	5475 5850 5475 5925
+Wire Wire Line
+	5800 5800 5800 5925
+Wire Wire Line
+	5900 5800 5900 5850
+Wire Wire Line
+	5900 5850 6100 5850
+Wire Wire Line
+	6100 5850 6100 5925
+Wire Wire Line
+	5475 6125 5475 6225
+Wire Wire Line
+	5475 6225 5550 6225
+Wire Wire Line
+	5475 6225 5350 6225
+Connection ~ 5475 6225
+Wire Wire Line
+	5800 6125 5800 6225
+Wire Wire Line
+	5800 6225 5750 6225
+Wire Wire Line
+	5800 6225 5875 6225
+Connection ~ 5800 6225
+Wire Wire Line
+	6100 6125 6100 6225
+Wire Wire Line
+	6100 6225 6075 6225
+Connection ~ 6100 6225
+Wire Wire Line
+	5150 6225 5075 6225
+Wire Wire Line
+	5075 6225 5075 6500
+$Comp
+L power:GND #PWR0111
+U 1 1 6137F787
+P 5075 6500
+F 0 "#PWR0111" H 5075 6250 50  0001 C CNN
+F 1 "GND" H 5075 6350 50  0000 C CNN
+F 2 "" H 5075 6500 50  0001 C CNN
+F 3 "" H 5075 6500 50  0001 C CNN
+	1    5075 6500
+	1    0    0    -1
+$EndComp
+Wire Wire Line
+	5700 5200 5700 5125
+Wire Wire Line
+	5700 5125 5800 5125
+Wire Wire Line
+	5900 5125 5900 5200
+Wire Wire Line
+	5800 5200 5800 5125
+Connection ~ 5800 5125
+Wire Wire Line
+	5800 5125 5900 5125
+Wire Wire Line
+	5700 5125 5600 5125
+Connection ~ 5700 5125
+$Comp
+L power:+3.3V #PWR0112
+U 1 1 613A0FD6
+P 5600 5025
+F 0 "#PWR0112" H 5600 4875 50  0001 C CNN
+F 1 "+3.3V" H 5600 5165 50  0000 C CNN
+F 2 "" H 5600 5025 50  0001 C CNN
+F 3 "" H 5600 5025 50  0001 C CNN
+	1    5600 5025
+	1    0    0    -1
+$EndComp
+Wire Wire Line
+	5600 5025 5600 5125
+Text Label 6825 6225 2    60   ~ 12
+DIP_SWITCH
+Wire Wire Line
+	6100 6225 6825 6225
+Text Label 3950 2650 0    60   ~ 12
+DIP_SWITCH
 NoConn ~ 7550 2650
+Wire Wire Line
+	3950 2650 4550 2650
 $EndSCHEMATC
