File: Base_board/battery_monitoring.sch (KiCad schematic (older format))
At the start: 22 parts, among them P1 TC_SWD, SW4 SW_SP3T, U7 STM32F030F4Px

Commit message: Fix older symbols assignation
Parts:
- C21, C22, C23, C24: symbol KXKM_audio_battery_module-rescue:C_Small -> Device:C_Small
- D10, D5, D6, D7, D8, D9: symbol KXKM_audio_battery_module-rescue:LED_Small -> Device:LED_Small
- P1: symbol KXKM_audio_battery_module-rescue:TC_SWD -> tom_kicad:TC_SWD
- R15, R16: symbol KXKM_audio_battery_module-rescue:R_Small -> Device:R_Small
- SW4: symbol KXKM_audio_battery_module-rescue:SW_SP3T -> Switch:SW_SP3T
- U7: symbol KXKM_audio_battery_module-rescue:STM32F030F4Px -> stm32:STM32F030F4Px
Changed lines of the file:
@@
 EESchema Schematic File Version 4
-LIBS:KXKM_audio_battery_module-cache
+LIBS:KXKM_ESP32_battery_management_board-cache
 EELAYER 29 0
 EELAYER END
@@
 $EndDescr
 $Comp
-L KXKM_audio_battery_module-rescue:STM32F030F4Px U7
+L stm32:STM32F030F4Px U7
 U 1 1 5A8AB82B
 P 6650 2050
@@
 $EndComp
 $Comp
-L KXKM_audio_battery_module-rescue:SW_SP3T SW4
+L Switch:SW_SP3T SW4
 U 1 1 5A8ABB36
 P 1150 5350
@@
 $EndComp
 $Comp
-L KXKM_audio_battery_module-rescue:TC_SWD P1
+L tom_kicad:TC_SWD P1
 U 1 1 5A9FA4FD
 P 1350 2050
@@
 ESP32_EN
 $Comp
-L KXKM_audio_battery_module-rescue:C_Small C23
+L Device:C_Small C23
 U 1 1 5AA0E0D5
 P 3000 3200
@@
 $EndComp
 $Comp
-L KXKM_audio_battery_module-rescue:C_Small C22
+L Device:C_Small C22
 U 1 1 5AA0E151
 P 2850 3200
@@
 $EndComp
 $Comp
-L KXKM_audio_battery_module-rescue:+3.3V #PWR084
+L power:+3.3V #PWR084
 U 1 1 5AA0E175
 P 2850 3000
@@
 Connection ~ 3350 3050
 $Comp
-L KXKM_audio_battery_module-rescue:GND #PWR085
+L power:GND #PWR085
 U 1 1 5AA0E1F8
 P 2850 3300
@@
 $EndComp
 $Comp
-L KXKM_audio_battery_module-rescue:GND #PWR086
+L power:GND #PWR086
 U 1 1 5AA0E21F
 P 3000 3300
@@
 $EndComp
 $Comp
-L KXKM_audio_battery_module-rescue:GND #PWR087
+L power:GND #PWR087
 U 1 1 5AA0E254
 P 9900 3000
@@
 USART1 is also used by\nthe serial bootloader.
 $Comp
-L KXKM_audio_battery_module-rescue:+BATT #PWR088
+L power:+BATT #PWR088
 U 1 1 5AA0E847
 P 1000 6650
@@
 Battery voltage measurement\n+BATT = 30V => 3.14V
 $Comp
-L KXKM_audio_battery_module-rescue:GND #PWR089
+L power:GND #PWR089
 U 1 1 5AA0EDE2
 P 1000 7250
@@
 $EndComp
 $Comp
-L KXKM_audio_battery_module-rescue:R_Small R15
+L Device:R_Small R15
 U 1 1 5AA0EE1E
 P 1000 6800
@@
 $EndComp
 $Comp
-L KXKM_audio_battery_module-rescue:R_Small R16
+L Device:R_Small R16
 U 1 1 5AA0EE4E
 P 1000 7100
@@
 VBAT_MEAS
 $Comp
-L KXKM_audio_battery_module-rescue:C_Small C21
+L Device:C_Small C21
 U 1 1 5AA0F3C7
 P 1250 7100
@@
 $EndComp
 $Comp
-L KXKM_audio_battery_module-rescue:GND #PWR090
+L power:GND #PWR090
 U 1 1 5AA0F425
 P 1250 7250
@@
 LED_BAR_4
 $Comp
-L KXKM_audio_battery_module-rescue:GND #PWR091
+L power:GND #PWR091
 U 1 1 5AA14FB1
 P 850 5400
@@
 NoConn ~ 1950 2150
 $Comp
-L KXKM_audio_battery_module-rescue:GND #PWR092
+L power:GND #PWR092
 U 1 1 5AA18D74
 P 750 2150
@@
 $EndComp
 $Comp
-L KXKM_audio_battery_module-rescue:+3.3V #PWR093
+L power:+3.3V #PWR093
 U 1 1 5AA18DFB
 P 750 1950
@@
 Li-Po\nLi-Fe\nCustom (set by ESP32)
 $Comp
-L KXKM_audio_battery_module-rescue:GND #PWR094
+L power:GND #PWR094
 U 1 1 5AA153F7
 P 10300 2450
@@
 Connection ~ 10150 2650
 $Comp
-L KXKM_audio_battery_module-rescue:C_Small C24
+L Device:C_Small C24
 U 1 1 5AA16056
 P 10150 2950
@@
 $EndComp
 $Comp
-L KXKM_audio_battery_module-rescue:GND #PWR095
+L power:GND #PWR095
 U 1 1 5AA1619D
 P 10150 3050
@@
 	2900 1450 3450 1450
 $Comp
-L KXKM_audio_battery_module-rescue:LED_Small D5
+L Device:LED_Small D5
 U 1 1 5AA7CC21
 P 6300 6900
@@
 $EndComp
 $Comp
-L KXKM_audio_battery_module-rescue:LED_Small D10
+L Device:LED_Small D10
 U 1 1 5AA7CEBB
 P 6650 6600
@@
 $EndComp
 $Comp
-L KXKM_audio_battery_module-rescue:LED_Small D6
+L Device:LED_Small D6
 U 1 1 5AA7CF29
 P 6300 7200
@@
 $EndComp
 $Comp
-L KXKM_audio_battery_module-rescue:LED_Small D7
+L Device:LED_Small D7
 U 1 1 5AA7CF73
 P 6650 7200
@@
 $EndComp
 $Comp
-L KXKM_audio_battery_module-rescue:LED_Small D9
+L Device:LED_Small D9
 U 1 1 5AA7CFBC
 P 6300 6600
@@
 $EndComp
 $Comp
-L KXKM_audio_battery_module-rescue:LED_Small D8
+L Device:LED_Small D8
 U 1 1 5AA7D01E
 P 6650 6900
@@
 $EndComp
 $Comp
-L KXKM_audio_battery_module-rescue:+3.3V #PWR0124
+L power:+3.3V #PWR0124
 U 1 1 5C82C903
 P 5250 4450
@@
 	5250 4450 5250 4550
 $Comp
-L KXKM_audio_battery_module-rescue:GND #PWR0125
+L power:GND #PWR0125
 U 1 1 5C82DF24
 P 5250 5400

Commit message: Fix component values > pick n place convention
Parts:
- R15: value 270k,1% -> 270k/1%
- R16: value 31.6k,1% -> 31.6k/1%
- R28: value 10k,1% -> 10k/1%
Changed lines of the file:
@@
 P 1000 6800
 F 0 "R15" H 1030 6820 50  0000 L CNN
-F 1 "270k,1%" H 1030 6760 50  0000 L CNN
+F 1 "270k/1%" H 1030 6760 50  0000 L CNN
 F 2 "Resistor_SMD:R_0603_1608Metric" H 1000 6800 50  0001 C CNN
 F 3 "" H 1000 6800 50  0001 C CNN
@@
 P 1000 7100
 F 0 "R16" H 1030 7120 50  0000 L CNN
-F 1 "31.6k,1%" H 1030 7060 50  0000 L CNN
+F 1 "31.6k/1%" H 1030 7060 50  0000 L CNN
 F 2 "Resistor_SMD:R_0603_1608Metric" H 1000 7100 50  0001 C CNN
 F 3 "" H 1000 7100 50  0001 C CNN
@@
 P 5250 4700
 F 0 "R28" H 5320 4746 50  0000 L CNN
-F 1 "10k,1%" H 5320 4655 50  0000 L CNN
+F 1 "10k/1%" H 5320 4655 50  0000 L CNN
 F 2 "Resistor_SMD:R_0603_1608Metric" V 5180 4700 50  0001 C CNN
 F 3 "~" H 5250 4700 50  0001 C CNN
