File: Base_board/battery_monitoring.sch (KiCad schematic (older format))
At the start: 20 parts, among them P1 TC_SWD, SW4 SW_SP3T, U7 STM32F030F4Px

Commit message: rescue from cache
Parts:
- P1: symbol tom_kicad:TC_SWD -> KXKM_ESP32_battery_management_board-rescue:TC_SWD-tom_kicad
- U7: symbol stm32:STM32F030F4Px -> KXKM_ESP32_battery_management_board-rescue:STM32F030F4Px-stm32
Changed lines of the file:
@@
 $EndDescr
 $Comp
-L stm32:STM32F030F4Px U7
+L KXKM_ESP32_battery_management_board-rescue:STM32F030F4Px-stm32 U7
 U 1 1 5A8AB82B
 P 6650 2050
@@
 $EndComp
 $Comp
-L tom_kicad:TC_SWD P1
+L KXKM_ESP32_battery_management_board-rescue:TC_SWD-tom_kicad P1
 U 1 1 5A9FA4FD
 P 1350 2050

Commit message: update, etc
Connections:
- net TEMP_MEAS renamed AUTOBOOT_SENSE
Changed lines of the file:
@@
 Wire Wire Line
 	2900 2750 3450 2750
-Text Label 2900 1350 0    60   ~ 12
-TEMP_MEAS
+Text HLabel 2900 1350 0    60   Input ~ 12
+AUTOBOOT_SENSE
 $EndSCHEMATC
