File: Base_board/power.sch (KiCad schematic (older format))
At the start: 39 parts, among them J13 Wire pad, J14 Wire pad, J15 Wire pad, J16 Wire pad, J9 USB_A, Q6 2N7002, SW3 SW_Push, U3 MCP16331T-E/CH, U4 BTS50080-1TEA, U5 DC_DC_POL

Commit message: rescue from cache
Parts:
- C6: symbol Device:CP1_Small -> KXKM_ESP32_battery_management_board-rescue:CP1_Small-Device
- J9: symbol KXKM_ESP32_battery_management_board-rescue:USB_A-Connector -> KXKM_ESP32_battery_management_board-rescue:USB_A-Connector-KXKM_ESP32_battery_management_board-rescue
- U5: symbol tom_kicad:DC_DC_POL -> KXKM_ESP32_battery_management_board-rescue:DC_DC_POL-tom_kicad
Changed lines of the file:
@@
 Battery power output.\nMax 10A
 $Comp
-L tom_kicad:DC_DC_POL U5
+L KXKM_ESP32_battery_management_board-rescue:DC_DC_POL-tom_kicad U5
 U 1 1 5A9FAEA4
 P 8650 2350
@@
 $EndComp
 $Comp
-L Device:CP1_Small C6
+L KXKM_ESP32_battery_management_board-rescue:CP1_Small-Device C6
 U 1 1 5AA2FD90
 P 2150 1500
@@
 	6800 2500 6800 2450
 $Comp
-L KXKM_ESP32_battery_management_board-rescue:USB_A-Connector J9
+L KXKM_ESP32_battery_management_board-rescue:USB_A-Connector-KXKM_ESP32_battery_management_board-rescue J9
 U 1 1 5C7F21B9
 P 9800 4000

Commit message: update, etc
Parts:
- added C11: 1uF, Capacitor_SMD:C_0603_1608Metric, symbol Device:C_Small
- added D14: Zener/3V/300mW, Diode_SMD:D_SOD-323, symbol Device:D_Zener_Small
- added D15: 1N4148WT, Diode_SMD:D_SOD-523, symbol Diode:1N4148WT
- added J5: Conn_01x02, Connector_PinHeader_2.54mm:PinHeader_1x02_P2.54mm_Vertical, symbol Connector_Generic:Conn_01x02
- added R28: 470R, Resistor_SMD:R_0603_1608Metric, symbol Device:R_Small
- added R32: 47k, Resistor_SMD:R_0603_1608Metric, symbol Device:R_Small
Connections:
- net +BATT: now also J5.1 (Pin_1)
- net GND: now also D14.2 (A), R32.2
- net at C26.1, D1.1 (K), D4.1 (K)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: now also D15.1 (K)
- new net: J5.2 (Pin_2), R28.1
- new net: C11.2, D15.2 (A), R32.1
- new net AUTOBOOT_SENSE: C11.1, D14.1 (K), R28.2
Other:
- note added: "SENSE is connected to the STM32 and give status \nof AUTOBOOT/SENSE information.\nThe MCU uses either a falling edge IRQ or polling to \nget status of autoboot (connected / disconnected)\nThe 3.3V regulator starts automatically \nwhen the jumper is connected, thanks to the edge detector (C/R)"
- moved on the sheet: D1, D4
Changed lines of the file:
@@
 Wire Wire Line
 	3150 5350 3150 5450
-Wire Wire Line
-	2000 5450 2200 5450
-Wire Wire Line
-	2800 5450 3150 5450
 Connection ~ 3150 5450
 Wire Wire Line
@@
 L Diode:1N4148WT D4
 U 1 1 5C719D34
-P 2650 5450
-F 0 "D4" H 2650 5667 50  0000 C CNN
-F 1 "1N4148WT" H 2700 5600 50  0000 C CNN
-F 2 "Diode_SMD:D_SOD-523" H 2650 5275 50  0001 C CNN
-F 3 "https://www.diodes.com/assets/Datasheets/ds30396.pdf" H 2650 5450 50  0001 C CNN
-	1    2650 5450
+P 2800 5450
+F 0 "D4" H 2800 5667 50  0000 C CNN
+F 1 "1N4148WT" H 2850 5600 50  0000 C CNN
+F 2 "Diode_SMD:D_SOD-523" H 2800 5275 50  0001 C CNN
+F 3 "https://www.diodes.com/assets/Datasheets/ds30396.pdf" H 2800 5450 50  0001 C CNN
+	1    2800 5450
 	1    0    0    -1
 $EndComp
@@
 L Diode:1N4148WT D1
 U 1 1 5C71A033
-P 2350 5450
-F 0 "D1" H 2350 5233 50  0000 C CNN
-F 1 "1N4148WT" H 2400 5300 50  0000 C CNN
-F 2 "Diode_SMD:D_SOD-523" H 2350 5275 50  0001 C CNN
-F 3 "https://www.diodes.com/assets/Datasheets/ds30396.pdf" H 2350 5450 50  0001 C CNN
-	1    2350 5450
+P 2250 5450
+F 0 "D1" H 2250 5233 50  0000 C CNN
+F 1 "1N4148WT" H 2300 5300 50  0000 C CNN
+F 2 "Diode_SMD:D_SOD-523" H 2250 5275 50  0001 C CNN
+F 3 "https://www.diodes.com/assets/Datasheets/ds30396.pdf" H 2250 5450 50  0001 C CNN
+	1    2250 5450
 	-1   0    0    1
 $EndComp
 Wire Wire Line
 	2500 5450 2500 6750
-Connection ~ 2500 5450
 $Comp
 L Diode:1N4148WT D12
@@
 Wire Wire Line
 	3700 6850 3700 7150
+$Comp
+L Diode:1N4148WT D15
+U 1 1 612D42B3
+P 2575 4300
+F 0 "D15" H 2575 4517 50  0000 C CNN
+F 1 "1N4148WT" H 2625 4450 50  0000 C CNN
+F 2 "Diode_SMD:D_SOD-523" H 2575 4125 50  0001 C CNN
+F 3 "https://www.diodes.com/assets/Datasheets/ds30396.pdf" H 2575 4300 50  0001 C CNN
+	1    2575 4300
+	0    1    -1   0
+$EndComp
+Wire Wire Line
+	2100 5450 2000 5450
+Wire Wire Line
+	2400 5450 2500 5450
+Wire Wire Line
+	2500 5450 2575 5450
+Connection ~ 2500 5450
+Wire Wire Line
+	2950 5450 3150 5450
+Connection ~ 2575 5450
+Wire Wire Line
+	2575 5450 2650 5450
+Wire Wire Line
+	2175 3775 2175 3825
+Connection ~ 2175 3775
+Wire Wire Line
+	2575 3775 2575 4150
+Wire Wire Line
+	2175 3775 2575 3775
+Wire Wire Line
+	2175 3700 2175 3775
+Wire Wire Line
+	2175 4025 2175 4075
+$Comp
+L power:GND #PWR09
+U 1 1 612CF015
+P 2175 4075
+F 0 "#PWR09" H 2175 3825 50  0001 C CNN
+F 1 "GND" H 2175 3925 50  0000 C CNN
+F 2 "" H 2175 4075 50  0001 C CNN
+F 3 "" H 2175 4075 50  0001 C CNN
+	1    2175 4075
+	1    0    0    -1
+$EndComp
+Wire Wire Line
+	2175 3425 2625 3425
+Connection ~ 2175 3425
+Wire Wire Line
+	2175 3500 2175 3425
+$Comp
+L Device:R_Small R32
+U 1 1 612C1FFA
+P 2175 3925
+F 0 "R32" H 2205 3945 50  0000 L CNN
+F 1 "47k" H 2205 3885 50  0000 L CNN
+F 2 "Resistor_SMD:R_0603_1608Metric" H 2175 3925 50  0001 C CNN
+F 3 "" H 2175 3925 50  0001 C CNN
+	1    2175 3925
+	1    0    0    -1
+$EndComp
+$Comp
+L Device:C_Small C11
+U 1 1 612C144A
+P 2175 3600
+F 0 "C11" H 2185 3670 50  0000 L CNN
+F 1 "1uF" H 2185 3520 50  0000 L CNN
+F 2 "Capacitor_SMD:C_0603_1608Metric" H 2175 3600 50  0001 C CNN
+F 3 "" H 2175 3600 50  0001 C CNN
+	1    2175 3600
+	1    0    0    -1
+$EndComp
+Wire Wire Line
+	1325 3425 2175 3425
+Text HLabel 2625 3425 2    60   Output ~ 12
+AUTOBOOT_SENSE
+Wire Wire Line
+	1325 3425 1325 3475
+Connection ~ 1325 3425
+$Comp
+L Device:D_Zener_Small D14
+U 1 1 61291FAE
+P 1325 3575
+F 0 "D14" V 1275 3675 50  0000 C CNN
+F 1 "Zener/3V/300mW" V 1375 3975 50  0000 C CNN
+F 2 "Diode_SMD:D_SOD-323" V 1325 3575 50  0001 C CNN
+F 3 "" V 1325 3575 50  0001 C CNN
+	1    1325 3575
+	0    1    1    0
+$EndComp
+Wire Wire Line
+	1325 3350 1325 3425
+Wire Wire Line
+	1325 3675 1325 3750
+$Comp
+L power:GND #PWR07
+U 1 1 6129868D
+P 1325 3750
+F 0 "#PWR07" H 1325 3500 50  0001 C CNN
+F 1 "GND" H 1325 3600 50  0000 C CNN
+F 2 "" H 1325 3750 50  0001 C CNN
+F 3 "" H 1325 3750 50  0001 C CNN
+	1    1325 3750
+	1    0    0    -1
+$EndComp
+$Comp
+L Device:R_Small R28
+U 1 1 61291126
+P 1325 3250
+F 0 "R28" H 1355 3270 50  0000 L CNN
+F 1 "470R" H 1375 3200 50  0000 L CNN
+F 2 "Resistor_SMD:R_0603_1608Metric" H 1325 3250 50  0001 C CNN
+F 3 "" H 1325 3250 50  0001 C CNN
+	1    1325 3250
+	1    0    0    -1
+$EndComp
+Wire Wire Line
+	2575 4450 2575 5450
+Text Notes 1625 3175 0    60   ~ 12
+SENSE is connected to the STM32 and give status \nof AUTOBOOT/SENSE information.\nThe MCU uses either a falling edge IRQ or polling to \nget status of autoboot (connected / disconnected)\nThe 3.3V regulator starts automatically  \nwhen the jumper is connected, thanks to the edge detector (C/R)
+$Comp
+L power:+BATT #PWR08
+U 1 1 6128D4C1
+P 1325 2625
+F 0 "#PWR08" H 1325 2475 50  0001 C CNN
+F 1 "+BATT" H 1325 2765 50  0000 C CNN
+F 2 "" H 1325 2625 50  0001 C CNN
+F 3 "" H 1325 2625 50  0001 C CNN
+	1    1325 2625
+	1    0    0    -1
+$EndComp
+$Comp
+L Connector_Generic:Conn_01x02 J5
+U 1 1 612FA68D
+P 925 2825
+F 0 "J5" H 843 3042 50  0000 C CNN
+F 1 "Conn_01x02" H 843 2951 50  0000 C CNN
+F 2 "Connector_PinHeader_2.54mm:PinHeader_1x02_P2.54mm_Vertical" H 925 2825 50  0001 C CNN
+F 3 "~" H 925 2825 50  0001 C CNN
+	1    925  2825
+	-1   0    0    -1
+$EndComp
+Wire Wire Line
+	1125 2825 1325 2825
+Wire Wire Line
+	1325 2625 1325 2825
+Wire Wire Line
+	1125 2925 1325 2925
+Wire Wire Line
+	1325 2925 1325 3150
 $EndSCHEMATC
