File: Base_board/KXKM_ESP32_battery_management_board.kicad_pcb (KiCad board)
At the start: 2 copper layers, 56.5 x 57.5 mm, 97 parts, among them J1 Conn_01x06, J11 TEST_1P, J13 Wire pad, J14 Wire pad, J15 Wire pad, J16 Wire pad, J2 TEST_1P, J3 Conn_02x10_Odd_Even, J4 Conn_01x04, J6 Conn_01x03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

Commit message: update, etc
Parts:
- removed REF**: SW_DIP_SPSTx03_Piano_CTS_Series194-3MSTN_W7.62mm_P2.54mm, Button_Switch_THT:SW_DIP_SPSTx03_Piano_CTS_Series194-3MSTN_W7.62mm_P2.54mm
- added C11: 1uF, Capacitor_SMD:C_0603_1608Metric, F.Cu at (151.5, 99.3)
- added D14: Zener/3V/300mW, Diode_SMD:D_SOD-323, F.Cu at (151.0, 101.9)
- added D15: 1N4148WT, Diode_SMD:D_SOD-523, F.Cu at (153.4, 96.6)
- added J5: Conn_01x02, Connector_PinHeader_2.54mm:PinHeader_1x02_P2.54mm_Vertical, F.Cu at (142.3, 133.9)
- added R28: 470R, Resistor_SMD:R_0603_1608Metric, F.Cu at (157.9, 109.7)
- added R32: 47k, Resistor_SMD:R_0603_1608Metric, F.Cu at (150.4, 97.6)
- added R33: 22k, Resistor_SMD:R_0603_1608Metric, F.Cu at (124.2, 90.3)
- added R34: 22k, Resistor_SMD:R_0603_1608Metric, F.Cu at (124.2, 91.9)
- added R35: 10k, Resistor_SMD:R_0603_1608Metric, F.Cu at (124.2, 88.6)
- added R36: 22k, Resistor_SMD:R_0603_1608Metric, F.Cu at (124.2, 83.7)
- added R37: 10k, Resistor_SMD:R_0603_1608Metric, F.Cu at (124.2, 85.3)
- added R38: 22k, Resistor_SMD:R_0603_1608Metric, F.Cu at (124.2, 87.0)
- added SW2: SW_DIP_x03, Button_Switch_THT:SW_DIP_SPSTx03_Piano_CTS_Series194-3MSTN_W7.62mm_P2.54mm, F.Cu at (133.6, 82.4)
- moved R25 7.28 mm to (131.1, 99.7)
- moved J2 6.58 mm to (121.7, 93.0)
- moved R23 4.39 mm to (124.6, 93.5)
- moved R27 4.22 mm to (124.6, 99.9)
- moved C24 4.21 mm to (124.6, 95.1)
- moved R26 4.14 mm to (124.6, 98.3)
- moved C22 4.05 mm to (124.6, 96.7)
- moved R24 3.74 mm to (127.9, 99.7), turned to 180 degrees
- moved D1 2.65 mm to (153.4, 93.5)
- moved D4 2.65 mm to (153.4, 95.0)
- moved R1 2.65 mm to (151.4, 94.3)
- moved R7 1.23 mm to (135.8, 112.2)
- moved SW1 0.62 mm to (109.6, 93.3)
- moved P1 0.24 mm to (108.6, 87.7)
- moved U4 0.16 mm to (146.2, 128.6)
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Connections:
- U1 pad 6: (no net) -> /DIP_SWITCH
- U7 pad 10: (no net) -> /Battery monitoring/AUTOBOOT_SENSE
Routing:
- net +BATT: track 0.00 -> 73.8 mm, vias 0 -> 2
- net VBUS: track 0.00 -> 56.5 mm
- net +3V3: track 0.00 -> 49.5 mm, vias 0 -> 3
- net +VSW: track 0.00 -> 46.3 mm
- net +BATT_RAW: track 0.00 -> 25.4 mm, vias 0 -> 6
- removed copper zone on B.Cu, net +BATT_RAW
- removed copper zone on F.Cu, net +BATT_RAW
- removed copper zone on B.Cu, net +VSW
Other:
- copper layers 2 -> 4
- board text removed: "A B -"

Commit message: passing drc
Parts:
- moved R9 13.1 mm to (147.3, 82.8), turned to 270 degrees
- moved C26 12.0 mm to (144.3, 81.6)
- moved R10 12.0 mm to (148.1, 85.1), turned to 0 degrees
- moved C8 10.2 mm to (148.9, 82.8), turned to 270 degrees
- moved C4 6.54 mm to (138.8, 93.9)
- moved C5 6.54 mm to (138.8, 91.4)
- moved U3 6.34 mm to (144.6, 84.3)
- moved D3 5.05 mm to (146.0, 89.8), turned to 0 degrees
- moved C7 4.93 mm to (144.2, 87.0), turned to 180 degrees
- moved D12 4.72 mm to (147.2, 87.0), turned to 0 degrees
- moved C9 2.93 mm to (140.3, 82.5), turned to 90 degrees
- moved L1 2.28 mm to (139.4, 87.4)
- moved C10 0.82 mm to (138.3, 82.5), turned to 90 degrees
- moved R26 0.58 mm to (124.0, 98.2)
- moved C22 0.52 mm to (124.1, 96.7)
Routing:
- net +3V3: track 49.5 -> 209.5 mm, vias 3 -> 14
- net /ESP32_EN: track 0.00 -> 65.1 mm, vias 0 -> 7
- net /LED_DATA_2: track 0.00 -> 59.9 mm, vias 0 -> 4
- net /LED_DATA_1: track 0.00 -> 52.6 mm, vias 0 -> 3
- net Net-(D10-Pad2): track 0.00 -> 43.7 mm, vias 0 -> 3
- net /Battery monitoring/AUTOBOOT_SENSE: track 0.00 -> 41.6 mm
- net /Battery monitoring/LOAD_I_SENSE: track 0.00 -> 40.7 mm, vias 0 -> 3
- net /DIP_SWITCH: track 0.00 -> 38.9 mm, vias 0 -> 2
- net /I2C_SDA: track 0.00 -> 37.9 mm, vias 0 -> 2
- net /ESP32_TXO: track 0.00 -> 36.9 mm, vias 0 -> 4
- net /Battery monitoring/EN_PUSH_BUTTON: track 0.00 -> 36.4 mm, vias 0 -> 3
- net /PROG_RTS: track 0.00 -> 36.3 mm, vias 0 -> 2
- net /I2C_SCL: track 0.00 -> 36.0 mm, vias 0 -> 2
- net +BATT: track 73.8 -> 109.0 mm, vias 2 -> 3
- net Net-(D10-Pad1): track 0.00 -> 35.1 mm, vias 0 -> 5
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- added copper zone on In1.Cu, net GND
- added copper zone on In2.Cu, net GND
Other:
- board text added: "BATT OUT < 10A"
- board text added: "DMX Gnd B A"
- board text added: "autoboot"
- board text added: "v3.0 09/2021"
- board text removed: "BATT OUT max 10A"
- board text removed: "DMX"
- board text removed: "v2.0 04/2019"

Commit message: releasing v3.0
Other:
- rule pad_to_mask_clearance: 0.07 -> 0
- board text added: "Dip Switch 3-positions"
- board text added: "V. Henry / Tom Magnier - v3.0 - 09/2021"
- board text removed: "T. Magnier - v2.0 - 04/2019"

Commit message: updating pcb
Routing:
- net +VSW: track 54.9 -> 96.9 mm, vias 1 -> 3
Changed lines of the file:
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@@
     (thickness 1.6)
     (drawings 180)
-    (tracks 903)
+    (tracks 917)
     (zones 0)
     (modules 109)
@@
   )
   (setup
-    (last_trace_width 0.15)
+    (last_trace_width 2)
     (user_trace_width 0.25)
     (user_trace_width 0.4)
@@
   (segment (start 144.090002 125.44) (end 138.5 125.44) (width 1.5) (layer F.Cu) (net 49))
   (segment (start 147.77 123.18) (end 146.350002 123.18) (width 1.5) (layer F.Cu) (net 49))
-  (segment (start 117.8 122.7) (end 113.5 127) (width 3) (layer In2.Cu) (net 49))
-  (segment (start 113.5 127) (end 113.5 135.25) (width 3) (layer In2.Cu) (net 49))
-  (segment (start 124.239999 124.739999) (end 122.2 122.7) (width 3) (layer In2.Cu) (net 49))
-  (segment (start 122.2 122.7) (end 117.8 122.7) (width 3) (layer In2.Cu) (net 49))
-  (segment (start 133.724001 124.739999) (end 124.239999 124.739999) (width 3) (layer In2.Cu) (net 49))
-  (segment (start 134.424002 125.44) (end 133.724001 124.739999) (width 3) (layer In2.Cu) (net 49))
-  (segment (start 138.5 125.44) (end 134.424002 125.44) (width 3) (layer In2.Cu) (net 49))
   (via (at 139.2 130.4) (size 0.6) (drill 0.3) (layers F.Cu B.Cu) (net 49))
-  (segment (start 139.2 126.14) (end 139.2 130.4) (width 2) (layer In2.Cu) (net 49))
-  (segment (start 138.5 125.44) (end 139.2 126.14) (width 2) (layer In2.Cu) (net 49))
   (segment (start 140.019999 131.280001) (end 142.04 131.280001) (width 2) (layer F.Cu) (net 49))
-  (segment (start 139.499999 130.760001) (end 140.019999 131.280001) (width 2) (layer F.Cu) (net 49))
+  (segment (start 139.499999 130.760001) (end 139.744999 131.005001) (width 2) (layer F.Cu) (net 49))
   (segment (start 139.499999 130.699999) (end 139.499999 130.760001) (width 2) (layer F.Cu) (net 49))
   (segment (start 139.2 130.4) (end 139.499999 130.699999) (width 2) (layer F.Cu) (net 49))
+  (segment (start 139.2 126.14) (end 139.2 129.7) (width 2) (layer B.Cu) (net 49))
+  (segment (start 138.5 125.44) (end 139.2 126.14) (width 2) (layer B.Cu) (net 49))
+  (segment (start 139.744999 131.005001) (end 140.019999 131.280001) (width 2) (layer F.Cu) (net 49))
+  (via (at 139.744999 131.005001) (size 0.6) (drill 0.3) (layers F.Cu B.Cu) (net 49))
+  (segment (start 139.2 129.7) (end 139.2 130.4) (width 2) (layer B.Cu) (net 49))
+  (via (at 139.2 129.7) (size 0.6) (drill 0.3) (layers F.Cu B.Cu) (net 49))
+  (segment (start 113.5 126.8) (end 117.510001 122.789999) (width 3) (layer In2.Cu) (net 49))
+  (segment (start 117.510001 122.789999) (end 122.589999 122.789999) (width 3) (layer In2.Cu) (net 49))
+  (segment (start 123.089999 122.789999) (end 125.039999 124.739999) (width 3) (layer In2.Cu) (net 49))
+  (segment (start 125.039999 124.739999) (end 135.639999 124.739999) (width 3) (layer In2.Cu) (net 49))
+  (segment (start 122.589999 122.789999) (end 123.089999 122.789999) (width 3) (layer In2.Cu) (net 49))
+  (segment (start 113.5 135.25) (end 113.5 126.969998) (width 3) (layer B.Cu) (net 49))
+  (segment (start 122.650001 123.119999) (end 122.869999 123.119999) (width 3) (layer B.Cu) (net 49))
+  (segment (start 122.320001 122.789999) (end 122.650001 123.119999) (width 3) (layer B.Cu) (net 49))
+  (segment (start 124.489999 124.739999) (end 137.799999 124.739999) (width 3) (layer B.Cu) (net 49))
+  (segment (start 137.799999 124.739999) (end 138.5 125.44) (width 3) (layer B.Cu) (net 49))
+  (segment (start 113.5 135.25) (end 113.5 126.8) (width 3) (layer In2.Cu) (net 49))
+  (segment (start 122.869999 123.119999) (end 124.489999 124.739999) (width 3) (layer B.Cu) (net 49))
+  (segment (start 117.679999 122.789999) (end 122.320001 122.789999) (width 3) (layer B.Cu) (net 49))
+  (segment (start 113.5 126.969998) (end 117.679999 122.789999) (width 3) (layer B.Cu) (net 49))
+  (segment (start 135.639999 124.739999) (end 138.139999 124.739999) (width 3) (layer In2.Cu) (net 49))
+  (segment (start 138.139999 124.739999) (end 139.4 126) (width 2) (layer In2.Cu) (net 49))
+  (segment (start 139.4 126) (end 139.4 130.8) (width 2) (layer In2.Cu) (net 49))
   (segment (start 116.1125 81.75) (end 114.7875 81.75) (width 0.25) (layer F.Cu) (net 50))
   (segment (start 110.3125 81.75) (end 108.9875 81.75) (width 0.25) (layer F.Cu) (net 50))
