File: Audio_board/KXKM_audio_board_for_ESP32.kicad_pcb (KiCad board)
At the start: 2 copper layers, 39.8 x 44.5 mm, 36 parts, among them J1 Conn_02x10_Odd_Even, J2 AudioJack2_Ground, J3 Conn_02x10_Odd_Even, J4 Conn_01x04, U1 DNP/TPS79133DBVR, U2 PCM5121, U3 Audio_amp_OEP30W, U4 Audio_amp_OEP30Wx2

Commit message: Fix component values > pick n place convention
Parts:
- C1: value DNP/0.1uF -> 0.1uF
- C10, C9: value 2.2uF,25V -> 2.2uF/25V
- C14: value 10uF,50V -> 10uF/50V
- C2: value DNP/10nF -> 10nF
- C3, C5: value 10uF,10V -> 10uF
- FB1: value 60R@100M -> Ferrite/60R/3A
- R1, R2: value 470R,1% -> 470R/1%
Changed lines of the file:
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@@
       (effects (font (size 1 1) (thickness 0.15)) (justify mirror))
     )
-    (fp_text value 2.2uF,25V (at 0 -1.43) (layer B.Fab) hide
+    (fp_text value 2.2uF/25V (at 0 -1.43) (layer B.Fab) hide
       (effects (font (size 1 1) (thickness 0.15)) (justify mirror))
     )
@@
       (effects (font (size 1 1) (thickness 0.15)) (justify mirror))
     )
-    (fp_text value 60R@100M (at 0 -1.65 270) (layer B.Fab) hide
+    (fp_text value Ferrite/60R/3A (at 0 -1.65 270) (layer B.Fab) hide
       (effects (font (size 1 1) (thickness 0.15)) (justify mirror))
     )
@@
       (effects (font (size 1 1) (thickness 0.15)) (justify mirror))
     )
-    (fp_text value 10uF,10V (at 0 -1.65) (layer B.Fab) hide
+    (fp_text value 10uF (at 0 -1.65) (layer B.Fab) hide
       (effects (font (size 1 1) (thickness 0.15)) (justify mirror))
     )
@@
       (effects (font (size 1 1) (thickness 0.15)) (justify mirror))
     )
-    (fp_text value 10uF,50V (at 0 -1.82 270) (layer B.Fab) hide
+    (fp_text value 10uF/50V (at 0 -1.82 270) (layer B.Fab) hide
       (effects (font (size 1 1) (thickness 0.15)) (justify mirror))
     )
@@
       (effects (font (size 1 1) (thickness 0.15)) (justify mirror))
     )
-    (fp_text value 470R,1% (at 0 -1.43 180) (layer B.Fab) hide
+    (fp_text value 470R/1% (at 0 -1.43 180) (layer B.Fab) hide
       (effects (font (size 1 1) (thickness 0.15)) (justify mirror))
     )
@@
       (effects (font (size 1 1) (thickness 0.15)) (justify mirror))
     )
-    (fp_text value 470R,1% (at 0 -1.43) (layer B.Fab) hide
+    (fp_text value 470R/1% (at 0 -1.43) (layer B.Fab) hide
       (effects (font (size 1 1) (thickness 0.15)) (justify mirror))
     )
@@
       (effects (font (size 1 1) (thickness 0.15)) (justify mirror))
     )
-    (fp_text value 2.2uF,25V (at 0 -1.43 90) (layer B.Fab) hide
+    (fp_text value 2.2uF/25V (at 0 -1.43 90) (layer B.Fab) hide
       (effects (font (size 1 1) (thickness 0.15)) (justify mirror))
     )
@@
       (effects (font (size 1 1) (thickness 0.15)) (justify mirror))
     )
-    (fp_text value 10uF,10V (at 0 -1.65 90) (layer B.Fab) hide
+    (fp_text value 10uF (at 0 -1.65 90) (layer B.Fab) hide
       (effects (font (size 1 1) (thickness 0.15)) (justify mirror))
     )
@@
       (effects (font (size 1 1) (thickness 0.15)) (justify mirror))
     )
-    (fp_text value DNP/10nF (at 0 -1.43 90) (layer B.Fab) hide
+    (fp_text value 10nF (at 0 -1.43 90) (layer B.Fab) hide
       (effects (font (size 1 1) (thickness 0.15)) (justify mirror))
     )
@@
       (effects (font (size 1 1) (thickness 0.15)) (justify mirror))
     )
-    (fp_text value DNP/0.1uF (at 0 -1.43 90) (layer B.Fab) hide
-      (effects (font (size 1 1) (thickness 0.15)) (justify mirror))
-    )
+    (fp_text value 0.1uF (at 0 -1.43 90) (layer B.Fab) hide
+      (effects (font (size 1 1) (thickness 0.15)) (justify mirror))
+    )
