File: Audio_board/KXKM_audio_board_for_ESP32.sch (KiCad schematic (older format))
At the start: 11 parts, among them J1 Conn_02x10_Odd_Even, J3 Conn_02x10_Odd_Even, U1 DNP/TPS79133DBVR

Commit message: Fix component values > pick n place convention
Parts:
- C1: value DNP/0.1uF -> 0.1uF
- C2: value DNP/10nF -> 10nF
- FB1: value 60R@100M -> Ferrite/60R/3A
Changed lines of the file:
@@
 P 6150 4050
 F 0 "FB1" V 5913 4050 50  0000 C CNN
-F 1 "60R@100M" V 6004 4050 50  0000 C CNN
+F 1 "Ferrite/60R/3A" V 6004 4050 50  0000 C CNN
 F 2 "Inductor_SMD:L_0805_2012Metric" V 6080 4050 50  0001 C CNN
 F 3 "~" H 6150 4050 50  0001 C CNN
@@
 P 7500 4250
 F 0 "C1" H 7408 4204 50  0000 R CNN
-F 1 "DNP/0.1uF" H 7408 4295 50  0000 R CNN
+F 1 "0.1uF" H 7408 4295 50  0000 R CNN
 F 2 "Capacitor_SMD:C_0603_1608Metric" H 7500 4250 50  0001 C CNN
 F 3 "~" H 7500 4250 50  0001 C CNN
@@
 P 8800 4350
 F 0 "C2" H 8708 4304 50  0000 R CNN
-F 1 "DNP/10nF" H 8708 4395 50  0000 R CNN
+F 1 "10nF" H 8708 4395 50  0000 R CNN
 F 2 "Capacitor_SMD:C_0603_1608Metric" H 8800 4350 50  0001 C CNN
 F 3 "~" H 8800 4350 50  0001 C CNN
