File: Remote_control_board/KXKM_esp_remote_control_module.kicad_pcb (KiCad board)
At the start: 2 copper layers, 48.9 x 70.8 mm, 21 parts, among them J1 Conn_01x03, J2 Conn_02x10_Odd_Even, J3 Conn_02x10_Odd_Even, J4 GPIOB_conn, J5 GPIOA_conn, J6 Conn_01x03, SW1 SW_SPDT, SW2 SW_Push, U1 HO10P-P-SP33, U3 MCP23017_SP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

Commit message: Add Gerbers
Other:
- board text added: "KXKM Remote board for ESP32 module V1.0"
Changed lines of the file:
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@@
   (general
     (thickness 1.6)
-    (drawings 50)
+    (drawings 51)
     (tracks 206)
     (zones 0)
@@
   (layers
     (0 F.Cu signal)
-    (31 B.Cu signal hide)
+    (31 B.Cu signal)
     (32 B.Adhes user)
     (33 F.Adhes user)
@@
   )
   (setup
-    (last_trace_width 1)
+    (last_trace_width 0.25)
     (user_trace_width 0.4)
     (user_trace_width 0.6)
@@
     )
   )
+  (gr_text "KXKM\nRemote board for\nESP32 module V1.0" (at 139.7 105.41 270) (layer F.SilkS)
+    (effects (font (size 0.8 0.8) (thickness 0.1)))
+  )
   (gr_line (start 156.972 99.568) (end 156.972 86.36) (layer F.SilkS) (width 0.2))
