File: Remote_control_board/KXKM_esp_remote_control_module.kicad_pcb (KiCad board)
At the start: 2 copper layers, 48.9 x 70.8 mm, 21 parts, among them J1 Conn_01x03, J2 Conn_02x10_Odd_Even, J3 Conn_02x10_Odd_Even, J4 GPIOB_conn, J5 GPIOA_conn, J6 Conn_01x03, SW1 SW_SPDT, SW2 SW_Push, U1 HO10P-P-SP33, U3 MCP23017_SP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

Commit message: update gerber and add current sensor doc
Parts:
- added D2: DIODE, Diode_SMD:D_0805_2012Metric_Pad1.15x1.40mm_HandSolder, F.Cu at (164.3, 100.3)
- moved C4 1.78 mm to (161.3, 102.6)
Connections:
- C4 pad 1: +3V3 -> Net-(C4-Pad1)
- U4 pad 1: +3V3 -> Net-(C4-Pad1)
Routing:
- net Net-(C4-Pad1): track 0.00 -> 6.88 mm
- net /DMX_DE: track 0.00 -> 5.79 mm, vias 0 -> 1
- net /ADC: track 44.2 -> 49.5 mm, vias 2 -> 3
- net /I2S_DATA: track 0.00 -> 5.17 mm, vias 0 -> 1
- net /SPI_MOSI: track 0.00 -> 4.80 mm, vias 0 -> 1
- net /SPI_SCK: track 0.00 -> 4.72 mm, vias 0 -> 1
- net /SPI_MISO: track 0.00 -> 4.28 mm, vias 0 -> 1
- net +3V3: track 123.2 -> 127.0 mm, vias 0 -> 1
- net /I2C_SCL: track 31.0 -> 34.6 mm, vias 0 -> 1
- net /SPI_CS: track 0.00 -> 3.27 mm, vias 0 -> 1
- net /I2S_BCK: track 0.00 -> 3.20 mm, vias 0 -> 1
- net /LED_D2: track 0.00 -> 3.13 mm, vias 0 -> 1
- net VBUS: track 57.0 -> 59.9 mm, vias 1 -> 2
- net /LED_D1: track 0.00 -> 2.87 mm, vias 0 -> 1
- net /DMX_RO: track 0.00 -> 2.75 mm, vias 0 -> 1
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Other:
- board size 48.9 x 70.8 mm -> 49.1 x 70.8 mm
