File: Remote_control_board/KXKM_esp_remote_control_module.sch (KiCad schematic (older format))
At the start: 21 parts, among them J1 Conn_01x03, J2 Conn_02x10_Odd_Even, J3 Conn_02x10_Odd_Even, J4 GPIOB_conn, J5 GPIOA_conn, J6 Conn_01x03, SW1 SW_SPDT, SW2 SW_Push, U1 HO10P-P-SP33, U3 MCP23017_SP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

Commit message: update gerber and add current sensor doc
Parts:
- added D2: DIODE, Diode_SMD:D_0805_2012Metric_Pad1.15x1.40mm_HandSolder, symbol pspice:DIODE
Connections:
- wire segments 157 -> 158
Changed lines of the file:
@@
 L power:+3.3V #PWR0112
 U 1 1 5E553F79
-P 9300 4300
-F 0 "#PWR0112" H 9300 4150 50  0001 C CNN
-F 1 "+3.3V" H 9315 4473 50  0000 C CNN
-F 2 "" H 9300 4300 50  0001 C CNN
-F 3 "" H 9300 4300 50  0001 C CNN
-	1    9300 4300
+P 9300 4150
+F 0 "#PWR0112" H 9300 4000 50  0001 C CNN
+F 1 "+3.3V" H 9315 4323 50  0000 C CNN
+F 2 "" H 9300 4150 50  0001 C CNN
+F 3 "" H 9300 4150 50  0001 C CNN
+	1    9300 4150
 	1    0    0    -1
 $EndComp
@@
 	0    1    1    0
 $EndComp
-Wire Wire Line
-	9300 4300 9300 4850
-Connection ~ 9300 4850
 $Comp
 L power:GND #PWR0114
@@
 Wire Wire Line
 	9000 3400 8850 3400
+$Comp
+L pspice:DIODE D2
+U 1 1 5E66F24C
+P 9300 4450
+F 0 "D2" V 9346 4322 50  0000 R CNN
+F 1 "DIODE" V 9255 4322 50  0000 R CNN
+F 2 "Diode_SMD:D_0805_2012Metric_Pad1.15x1.40mm_HandSolder" H 9300 4450 50  0001 C CNN
+F 3 "" H 9300 4450 50  0001 C CNN
+	1    9300 4450
+	0    -1   -1   0
+$EndComp
+Wire Wire Line
+	9300 4650 9300 4850
+Connection ~ 9300 4850
+Wire Wire Line
+	9300 4250 9300 4150
 $EndSCHEMATC
