File: Base_board/in-progress/battery_monitoring.kicad_sch (KiCad schematic)
At the start: 20 parts, among them P1 TC_SWD, SW4 SW_SP3T, U7 STM32F030F4Px

Commit message: update v3.2
-  connecteur XT60 coudé (et disponible chez JLCPCB)
- modification de l’autoboot pour un redémarrage en cas de perte brêve d’alimentation,
- ajout de l’empreinte pour rajouter une lecteur microSD
- mise à jour des piste de sortie batterie conforme pour 10A
- suppression des pin I2C (déjà dispo sur le GPIO)
- connecteur JST B3B-EH pour un câblage et éviter les soudure qui casse sur les sortie pour LED
- ESP32 en version 16M
Parts:
- C22, C23, C24: LCSC (none) -> C14663
- D10: LCSC (none) -> C2286
- D5, D6, D7: LCSC (none) -> C72043
- D8, D9: LCSC (none) -> C72038
- R15: LCSC (none) -> C22965
- R16: LCSC (none) -> C25967
- R23: LCSC (none) -> C21190
- R24, R25, R26, R27: LCSC (none) -> C22775
- SW4: LCSC (none) -> C160878
- U7: value STM32F030F4Px -> STM32F070F6Px; LCSC (none) -> C86951
Other:
- title: (none) -> ESP32 battery management module

Commit message: update to v3.2 and casing 3D View
Other:
- company: (none) -> for : KXKM
Changed lines of the file:
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@@
     (date "2023-06-14")
     (rev "3.2")
-    (comment 1 "Tom Magnier / initial release")
-    (comment 2 "Viven Henry / SD, Switch, Autoboot")
-    (comment 3 "Clément SAILLANT / update Autoboot, readd SD")
+    (company "for : KXKM")
+    (comment 1 "update PCB, add optional SD, ....")
+    (comment 2 "Clément SAILLANT (v3.2) : improve Autoboot")
+    (comment 3 "Viven Henry (v3) : remove SD, add Switch, add Autoboot")
+    (comment 4 "Tom Magnier :  initial release (v1 & v2)")
   )
   (junction (at 31.75 176.53) (diameter 0) (color 0 0 0 0)
