File: Base_board/v3.2/KXKM_ESP32_battery_management_board.kicad_pcb (KiCad board)
At the start: 4 copper layers, 56.5 x 57.5 mm, 110 parts, among them J1 Conn_01x06, J10 XT60PW-M, J11 TEST_1P, J12 Conn_01x02_Socket, J15 Wire pad, J16 Wire pad, J2 TEST_1P, J3 Conn_02x10_Odd_Even, J4 112J-TDAR-R01, J5 Conn_01x02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

Commit message: last order
Parts:
- J3: footprint Connector_PinSocket_2.54mm:PinSocket_2x10_P2.54mm_Vertical_SMD -> easyeda2kicad:HDR-SMD_20P-P2.54-V-F-R2-C10-S2.54-LS7.2-1
- SW1: footprint Button_Switch_SMD:SW_SPST_KMR2 -> easyeda2kicad:SW-SMD_L3.0-W2.0-LS3.5
- SW3: footprint Button_Switch_THT:SW_Tactile_SPST_Angled_PTS645Vx31-2LFS -> easyeda2kicad:KEY-TH_TC-6615-5.5-160G
- moved SW3 2.55 mm to (154.5, 84.4), turned to 180 degrees
Routing:
- net +3V3: track 222.9 -> 227.2 mm
- net GND: track 15.7 -> 14.1 mm, vias 22 -> 20
